Commit message: fixup the robot description for dingo o

File: dingo_description/urdf/dingo-o.urdf.xacro (robot description, xacro)
@@ -1,4 +1,8 @@
 <?xml version="1.0"?>
 <robot name="dingo" xmlns:xacro="http://www.ros.org/wiki/xacro">
+	<!-- Enable setting arguments from the launch file -->
+  <xacro:arg name="physical_robot" default="true"/>
+	<xacro:property name="control_empty_default" value="" />
+	<xacro:arg name="control_yaml_file" default="$(control_empty_default)"/>
   <xacro:property name="PI" value="3.1415926535897931" />
   <xacro:property name="wheelbase" value="0.570" />
@@ -89,5 +93,5 @@
       <origin xyz="0 0 0" rpy="0 0 0"/>
       <mass value="14"/>
-      <!-- Moments of inertia: ( chassis without wheels ) -->
+      <!-- Moments of inertia ( chassis without wheels ) -->
       <inertia
         ixx="0.35498" ixy="0" ixz="0"
@@ -173,7 +177,43 @@
     <child link="front_bumper_mount" />
   </joint>
+	<!-- ROS 2 control -->
+	<ros2_control name="dingo-o_hardware" type="system">
+		<hardware>
+			<xacro:if value="$(arg physical_robot)">
+				<plugin>dingo_base/DingoHardware</plugin>
+				<param name="gear_ratio">24</param>
+				<param name="canbus_dev">can0</param>
+				<param name="encoder_cpr">10</param>
+				<param name="flip_motor_direction">0</param> <!-- 1/0 instead of true/false -->
+				<param name="gains_p">0.025</param>
+				<param name="gains_i">0.005</param>
+				<param name="gains_d">0.0</param>
+			</xacro:if>
+			<xacro:unless value="$(arg physical_robot)">
+				<plugin>gazebo_ros2_control/GazeboSystem</plugin>
+			</xacro:unless>
+		</hardware>
+		<joint name="left_wheel">
+			<command_interface name="velocity">
+				<param name="min">-10</param>
+				<param name="max">10</param>
+			</command_interface>
+			<state_interface name="position"/>
+			<state_interface name="velocity"/>
+		</joint>
+		<joint name="right_wheel">
+			<command_interface name="velocity">
+				<param name="min">-10</param>
+				<param name="max">10</param>
+			</command_interface>
+			<state_interface name="position"/>
+			<state_interface name="velocity"/>
+		</joint>
+	</ros2_control>
   <!-- Bring in simulation data for Gazebo. -->
   <xacro:include filename="$(find dingo_description)/urdf/dingo.gazebo" />
-  <xacro:include filename="$(find dingo_description)/urdf/dingo-o.gazebo" />
+	<xacro:unless value="$(arg physical_robot)">
+		<xacro:include filename="$(find dingo_description)/urdf/dingo-o.gazebo" />
+	</xacro:unless>
   <!-- Optional standard accessories, including their simulation data. The rendering
        of these into the final description is controlled by optenv variables, which

Commit message: changes for dingo o

File: dingo_description/urdf/dingo-o.urdf.xacro (robot description, xacro)
@@ -1,8 +1,8 @@
 <?xml version="1.0"?>
 <robot name="dingo" xmlns:xacro="http://www.ros.org/wiki/xacro">
-	<!-- Enable setting arguments from the launch file -->
+  <!-- Enable setting arguments from the launch file -->
   <xacro:arg name="physical_robot" default="true"/>
-	<xacro:property name="control_empty_default" value="" />
-	<xacro:arg name="control_yaml_file" default="$(control_empty_default)"/>
+  <xacro:property name="control_empty_default" value="" />
+  <xacro:arg name="control_yaml_file" default="${control_empty_default}"/>
   <xacro:property name="PI" value="3.1415926535897931" />
   <xacro:property name="wheelbase" value="0.570" />
@@ -79,5 +79,5 @@
       <origin xyz="0 0 0" rpy="0 0 0"/>
       <geometry>
-        <mesh filename="file://$(find dingo_description)/meshes/omni_chassis.dae"/>
+        <mesh filename="package://dingo_description/meshes/omni_chassis.dae"/>
       </geometry>
       <material name="dark_grey" />
@@ -86,5 +86,5 @@
       <origin xyz="0 0 0"/>
       <geometry>
-        <mesh filename="file://$(find dingo_description)/meshes/omni_chassis_collision.stl"/>
+        <mesh filename="package://dingo_description/meshes/omni_chassis_collision.stl"/>
       </geometry>
     </collision>
@@ -177,43 +177,59 @@
     <child link="front_bumper_mount" />
   </joint>
-	<!-- ROS 2 control -->
-	<ros2_control name="dingo-o_hardware" type="system">
-		<hardware>
-			<xacro:if value="$(arg physical_robot)">
-				<plugin>dingo_base/DingoHardware</plugin>
-				<param name="gear_ratio">24</param>
-				<param name="canbus_dev">can0</param>
-				<param name="encoder_cpr">10</param>
-				<param name="flip_motor_direction">0</param> <!-- 1/0 instead of true/false -->
-				<param name="gains_p">0.025</param>
-				<param name="gains_i">0.005</param>
-				<param name="gains_d">0.0</param>
-			</xacro:if>
-			<xacro:unless value="$(arg physical_robot)">
-				<plugin>gazebo_ros2_control/GazeboSystem</plugin>
-			</xacro:unless>
-		</hardware>
-		<joint name="left_wheel">
-			<command_interface name="velocity">
-				<param name="min">-10</param>
-				<param name="max">10</param>
-			</command_interface>
-			<state_interface name="position"/>
-			<state_interface name="velocity"/>
-		</joint>
-		<joint name="right_wheel">
-			<command_interface name="velocity">
-				<param name="min">-10</param>
-				<param name="max">10</param>
-			</command_interface>
-			<state_interface name="position"/>
-			<state_interface name="velocity"/>
-		</joint>
-	</ros2_control>
+  <!-- ROS 2 control -->
+  <ros2_control name="dingo-o_hardware" type="system">
+    <hardware>
+      <xacro:if value="$(arg physical_robot)">
+        <plugin>dingo_base/DingoHardware</plugin>
+        <param name="gear_ratio">24</param>
+        <param name="canbus_dev">vcan0</param>
+        <param name="encoder_cpr">10</param>
+        <param name="flip_motor_direction">0</param> <!-- 1/0 instead of true/false -->
+        <param name="gains_p">0.025</param>
+        <param name="gains_i">0.005</param>
+        <param name="gains_d">0.0</param>
+      </xacro:if>
+      <xacro:unless value="$(arg physical_robot)">
+        <plugin>gazebo_ros2_control/GazeboSystem</plugin>
+      </xacro:unless>
+    </hardware>
+    <joint name="front_left_wheel">
+      <command_interface name="velocity">
+        <param name="min">-10</param>
+        <param name="max">10</param>
+      </command_interface>
+      <state_interface name="position"/>
+      <state_interface name="velocity"/>
+    </joint>
+    <joint name="front_right_wheel">
+      <command_interface name="velocity">
+        <param name="min">-10</param>
+        <param name="max">10</param>
+      </command_interface>
+      <state_interface name="position"/>
+      <state_interface name="velocity"/>
+    </joint>
+    <joint name="rear_left_wheel">
+      <command_interface name="velocity">
+        <param name="min">-10</param>
+        <param name="max">10</param>
+      </command_interface>
+      <state_interface name="position"/>
+      <state_interface name="velocity"/>
+    </joint>
+    <joint name="rear_right_wheel">
+      <command_interface name="velocity">
+        <param name="min">-10</param>
+        <param name="max">10</param>
+      </command_interface>
+      <state_interface name="position"/>
+      <state_interface name="velocity"/>
+    </joint>
+  </ros2_control>
   <!-- Bring in simulation data for Gazebo. -->
   <xacro:include filename="$(find dingo_description)/urdf/dingo.gazebo" />
-	<xacro:unless value="$(arg physical_robot)">
-		<xacro:include filename="$(find dingo_description)/urdf/dingo-o.gazebo" />
-	</xacro:unless>
+  <xacro:unless value="$(arg physical_robot)">
+    <xacro:include filename="$(find dingo_description)/urdf/dingo-o.gazebo" />
+  </xacro:unless>
   <!-- Optional standard accessories, including their simulation data. The rendering
        of these into the final description is controlled by optenv variables, which
